File: src/chip8.kicad_sch (KiCad schematic)
At the start: 43 parts, among them J1 204926-1103, M1 STM32L476RGT6, Q1 DMP2240UW-7, Q2 BC847-T, T1 5002, T2 5002, T3 5002, T4 5002, U1 MCP73831T-2ACI_OT, U2 PCM12SMTR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

Commit message: ground plane and corrections done
Parts:
- added BAT1: Battery, symbol Device:Battery
- added batt1: Conn_01x02_Pin, Connector_PinSocket_2.54mm:PinSocket_1x02_P2.54mm_Vertical, symbol Connector:Conn_01x02_Pin
- renumbered aaaa1 to buzz1
Connections:
- net GND: now also batt1.2 (Pin_2)
- net VBAT1: now also batt1.1 (Pin_1)
